File: HF103-ADC.kicad_sch (KiCad schematic)
At the start: 19 parts, among them T1 ETC1-1T-2TR, U4 LTC2208CUP-14-PBF

Commit message: Commit latest schematic changes
Parts:
- removed T1: ETC1-1T-2TR, MACOM_ETC1-1T-2TR:ETC1-1-13TR_MCM, symbol MACOM_ETC1-1T-2TR:ETC1-1T-2TR
- added C19 (x3): 0.1uF, Capacitor_SMD:C_0805_2012Metric_Pad1.18x1.45mm_HandSolder, symbol Device:C
- added TR1: ETC1-1-13, Transformer_SMD:Transformer_MACOM_SM-22, symbol Transformer:ETC1-1-13
- C19: value 8p2 -> 8.2pF
- C19: value 8p2 -> 0.1uF
- C19: value 4p2 -> 0.1uF
- R14, R15: value 100 -> 50
Connections:
- net CLK0: now also C19.2
- net GND: now also C19.2, C19.2
- net at C19.1, R1.1, R14.1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: now also TR1.1
- net at C19.2, R1.2, R15.2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: now also TR1.5
- net at C19.1: now also TR1.2
- new net: C19.1, TR1.3
- no-connect marks 1 -> 20
Other:
- note added: "Pin 65 (Back) is Gnd-soldered to PC"
- note added: "Pins for 16bit part"
- moved on the sheet: C19, C20, L6, L7, R1, R14, R15, R5, U4
