File: HF103-Power.kicad_sch (KiCad schematic)
At the start: 19 parts, among them J1 Barrel_Jack, P8 Conn_01x03, U1 AP7361C-33E, U6 AMS1117CD-1.8, U7 NCP360SNT1G

Commit message: Commit latest schematic changes
Connections:
- net GND: now also NT1.1
Changed lines of the file:
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@@
     (stroke (width 0) (type default))
   )
-  (wire (pts (xy 60.96 73.66) (xy 67.31 73.66))
+  (wire (pts (xy 63.5 73.66) (xy 67.31 73.66))
     (stroke (width 0) (type default))
   )
@@
     (stroke (width 0) (type default))
   )
-  (wire (pts (xy 60.96 67.31) (xy 60.96 73.66))
+  (wire (pts (xy 63.5 76.2) (xy 63.5 73.66))
     (stroke (width 0) (type default))
   )
@@
         )
       )
+    )
+  )
+  (symbol (lib_id "power:GND") (at 63.5 76.2 0) (unit 1)
+    (in_bom yes) (on_board yes) (dnp no)
+    (property "Reference" "#PWR043" (at 63.5 82.55 0)
+      (effects (font (size 1.27 1.27)) hide)
+    )
+    (property "Value" "GND" (at 60.96 76.2 0)
+      (effects (font (size 1 1)))
+    )
+    (property "Footprint" "" (at 63.5 76.2 0)
+      (effects (font (size 1.27 1.27)) hide)
+    )
+    (property "Datasheet" "" (at 63.5 76.2 0)
+      (effects (font (size 1.27 1.27)) hide)
+    )
+    (pin "1")
+    (instances
+      (project "HF103-redux"
+        (path "/a6bdb5ae-8f9c-40cb-b68a-86d3cad405bf/8c380369-8e8f-45e8-9e3f-03ede4dd855a"
+          (reference "#PWR043") (unit 1)
+        )
+      )
