File: HF103-USB.kicad_sch (KiCad schematic)
At the start: 34 parts, among them J1 Conn_02x20_Odd_Even, J2 Conn_02x20_Odd_Even, J4 Conn_01x08, J5 Conn_01x04, P3 Conn_01x16

Commit message: Commit latest schematic changes
Connections:
- net at C21.1, C29.1, J4.5 (Pin_5)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: no longer C25.1, C30.1, J4.6 (Pin_6), P3.5 (Pin_5), R8.2
- new net: C25.1, C30.1, J4.6 (Pin_6), P3.5 (Pin_5), R8.2
